Commit message: Debug
Edited the package name

File: description/urdf/scooter.xacro (robot description, xacro)
@@ -67,5 +67,5 @@
         <visual>
         <geometry>
-            <mesh filename="package://scooter/description/meshes/frame.stl" scale="${scale} ${scale} ${scale}"/>
+            <mesh filename="package://autonomous-scooter/description/meshes/frame.stl" scale="${scale} ${scale} ${scale}"/>
         </geometry>
         <material name='black'/>
