Commit message: changed depth camera parent link to base_link

File: urdf/scooter.urdf.xacro (robot description, xacro)
@@ -22,5 +22,5 @@
         <inertia ixx="${steering_ixx}" ixy="${steering_ixy}" ixz="${steering_ixz}" iyy="${steering_iyy}" iyz="${steering_iyz}" izz="${steering_izz}"/>
     </link>
-        <joint name="front_wheel_to_steering_joint" type="revolute">
+        <joint name="base_to_steering_joint" type="revolute">
             <parent link="base_link"/>
             <child link="steering_link"/>
@@ -28,8 +28,9 @@
             <limit lower="-${pi/4}" upper="${pi/4}" effort="0.0" velocity="0.0"/>
             <axis xyz="0 0 1"/>
+            <limit effort="30" velocity="1.0"/>
         </joint>
-        <transmission name="tran1">
+        <!-- <transmission name="tran1">
             <type>transmission_interface/SimpleTransmission</type>
-            <joint name="front_wheel_to_steering_joint">
+            <joint name="base_to_steering_joint">
                 <hardwareInterface>hardware_interface/EffortJointInterface</hardwareInterface>
             </joint>
@@ -38,5 +39,5 @@
                 <mechanicalReduction>1</mechanicalReduction>
             </actuator>
-        </transmission>
+        </transmission> -->
     <!-- front wheel -->
     <link name="front_wheel_link">
@@ -57,13 +58,14 @@
         <inertia ixx="${front_ixx}" ixy="${front_ixy}" ixz="${front_ixz}" iyy="${front_iyy}" iyz="${front_iyz}" izz="${front_izz}"/>
     </link>
-        <joint name="base_to_front_joint" type="continuous">
+        <joint name="steering_to_front_joint" type="continuous">
             <parent link="steering_link"/>
             <child link="front_wheel_link"/>
             <origin xyz="0.0 0.0 -${steering_length/2}" rpy="0.0 0.0 0.0"/>
             <axis xyz="0 1 0"/>
+            <limit effort="50" velocity="2.0"/>
         </joint>
-        <transmission name="tran2">
+        <!-- <transmission name="tran2">
             <type>transmission_interface/SimpleTransmission</type>
-            <joint name="base_to_front_joint">
+            <joint name="steering_to_front_joint">
                 <hardwareInterface>hardware_interface/EffortJointInterface</hardwareInterface>
             </joint>
@@ -72,5 +74,5 @@
                 <mechanicalReduction>1</mechanicalReduction>
             </actuator>
-        </transmission>
+        </transmission> -->
     <!-- frame_link -->
     <link name="frame_link">
@@ -142,4 +144,5 @@
             <origin xyz="0 ${length_back_axis/2} 0.0" rpy="${pi/2} 0.0 0.0"/>
             <axis xyz="0 0 1"/>
+            <limit effort="50" velocity="2.0"/>
         </joint>
     <!-- back wheel right -->
@@ -166,9 +169,10 @@
             <origin xyz="0.0 -${length_back_axis / 2} 0.0" rpy="${pi/2} 0.0 0.0"/>
             <axis xyz="0 0 1"/>
+            <limit effort="50" velocity="2.0"/>
         </joint>
     <!-- depth camera -->
     <xacro:include filename="$(find autonomous-scooter)/urdf/realsense_urdf/_d435.urdf.xacro" />
-    <xacro:sensor_d435 parent="steering_link" use_nominal_extrinsics="false" add_plug="false" use_mesh="true">
-        <origin xyz="0.03 0 0.1" rpy="0 0 0"/>
+    <xacro:sensor_d435 parent="base_link" use_nominal_extrinsics="false" add_plug="false" use_mesh="true">
+        <origin xyz="0.03 0 0.3" rpy="0 0 0"/>
     </xacro:sensor_d435>
 </robot>
