Commit message: update

File: urdf/properties.xacro (robot description, xacro)
@@ -11,45 +11,53 @@
         <color rgba="0 0 0.8 0.7"/>
     </material>
+<!--     <inertial>
+        <origin xyz="0 0 0" rpy="0 0 0" />
+        <mass value="1" />
+        <inertia
+          ixx="1.0" ixy="0.0" ixz="0.0"
+          iyy="1.0" iyz="0.0"
+          izz="1.0" />
+    </inertial> -->
     <!-- xacro properties -->
     <xacro:property name="thick_wheel" value="0.044" />
         <!-- frame_link -->
     <xacro:property name="scale" value="${0.01}" />
-    <xacro:property name="mass_frame_link" value="0.0" />
-    <xacro:property name="front_ixx" value="0.0" />
-    <xacro:property name="front_ixy" value="0.0" />
-    <xacro:property name="front_ixz" value="0.0" />
-    <xacro:property name="front_iyy" value="0.0" />
-    <xacro:property name="front_iyz" value="0.0" />
-    <xacro:property name="front_izz" value="0.0" />
+    <xacro:property name="mass_frame_link" value="1.0" />
+    <xacro:property name="front_ixx" value="1.0" />
+    <xacro:property name="front_ixy" value="0.1" />
+    <xacro:property name="front_ixz" value="0.1" />
+    <xacro:property name="front_iyy" value="0.1" />
+    <xacro:property name="front_iyz" value="0.1" />
+    <xacro:property name="front_izz" value="0.1" />
         <!-- steering_link -->
     <xacro:property name="thick_steering" value="0.02" />
     <xacro:property name="alpha" value="${80 * pi / 180}" />
     <xacro:property name="steering_length" value="${0.2}" />
-    <xacro:property name="mass_steering_link" value="${0.0}" />
-    <xacro:property name="steering_ixx" value="0.0" />
-    <xacro:property name="steering_ixy" value="0.0" />
-    <xacro:property name="steering_ixz" value="0.0" />
-    <xacro:property name="steering_iyy" value="0.0" />
-    <xacro:property name="steering_iyz" value="0.0" />
-    <xacro:property name="steering_izz" value="0.0" />
+    <xacro:property name="mass_steering_link" value="${1.0}" />
+    <xacro:property name="steering_ixx" value="1.0" />
+    <xacro:property name="steering_ixy" value="0.1" />
+    <xacro:property name="steering_ixz" value="0.1" />
+    <xacro:property name="steering_iyy" value="0.1" />
+    <xacro:property name="steering_iyz" value="0.1" />
+    <xacro:property name="steering_izz" value="0.1" />
         <!-- front wheel  -->
     <xacro:property name="rad_front_wheel" value="${0.216/2}" />
-    <xacro:property name="mass_front_wheel" value="0.0" />
-    <xacro:property name="front_ixx" value="0.0" />
-    <xacro:property name="front_ixy" value="0.0" />
-    <xacro:property name="front_ixz" value="0.0" />
-    <xacro:property name="front_iyy" value="0.0" />
-    <xacro:property name="front_iyz" value="0.0" />
-    <xacro:property name="front_izz" value="0.0" />
+    <xacro:property name="mass_front_wheel" value="1.0" />
+    <xacro:property name="front_ixx" value="1.0" />
+    <xacro:property name="front_ixy" value="0.1" />
+    <xacro:property name="front_ixz" value="0.1" />
+    <xacro:property name="front_iyy" value="0.1" />
+    <xacro:property name="front_iyz" value="0.1" />
+    <xacro:property name="front_izz" value="0.1" />
         <!-- back axis -->
     <xacro:property name="length_back_axis" value="0.3" />
     <xacro:property name="rad_back_wheel" value="${0.203/2}" />
         <!-- back wheel inertia -->
-    <xacro:property name="mass_back_wheel" value="0.0" />
-    <xacro:property name="back_ixx" value="0.0" />
-    <xacro:property name="back_ixy" value="0.0" />
-    <xacro:property name="back_ixz" value="0.0" />
-    <xacro:property name="back_iyy" value="0.0" />
-    <xacro:property name="back_iyz" value="0.0" />
-    <xacro:property name="back_izz" value="0.0" />
+    <xacro:property name="mass_back_wheel" value="1.0" />
+    <xacro:property name="back_ixx" value="1.0" />
+    <xacro:property name="back_ixy" value="0.1" />
+    <xacro:property name="back_ixz" value="0.1" />
+    <xacro:property name="back_iyy" value="0.1" />
+    <xacro:property name="back_iyz" value="0.1" />
+    <xacro:property name="back_izz" value="0.1" />
 </robot>

File: urdf/scooter.urdf.xacro (robot description, xacro)
@@ -29,4 +29,14 @@
             <axis xyz="0 0 1"/>
         </joint>
+        <transmission name="tran1">
+            <type>transmission_interface/SimpleTransmission</type>
+            <joint name="front_wheel_to_steering_joint">
+                <hardwareInterface>hardware_interface/EffortJointInterface</hardwareInterface>
+            </joint>
+            <actuator name="steering_motor">
+                <hardwareInterface>hardware_interface/EffortJointInterface</hardwareInterface>
+                <mechanicalReduction>1</mechanicalReduction>
+            </actuator>
+        </transmission>
     <!-- front wheel -->
     <link name="front_wheel_link">
@@ -53,4 +63,14 @@
             <axis xyz="0 1 0"/>
         </joint>
+        <transmission name="tran2">
+            <type>transmission_interface/SimpleTransmission</type>
+            <joint name="base_to_front_joint">
+                <hardwareInterface>hardware_interface/EffortJointInterface</hardwareInterface>
+            </joint>
+            <actuator name="wheel_motor">
+                <hardwareInterface>hardware_interface/EffortJointInterface</hardwareInterface>
+                <mechanicalReduction>1</mechanicalReduction>
+            </actuator>
+        </transmission>
     <!-- frame_link -->
     <link name="frame_link">
@@ -152,4 +172,3 @@
         <origin xyz="0.03 0 0.1" rpy="0 0 0"/>
     </xacro:sensor_d435>
-    <!-- <gazebo reference="scooter"/> -->
 </robot>

Commit message: update

File: urdf/properties.xacro (robot description, xacro)
@@ -17,5 +17,5 @@
           ixx="1.0" ixy="0.0" ixz="0.0"
           iyy="1.0" iyz="0.0"
-          izz="1.0" />
+          izz="1.0 />
     </inertial> -->
     <!-- xacro properties -->
@@ -23,41 +23,41 @@
         <!-- frame_link -->
     <xacro:property name="scale" value="${0.01}" />
-    <xacro:property name="mass_frame_link" value="1.0" />
+    <xacro:property name="mass_frame_link" value="6.5" />
     <xacro:property name="front_ixx" value="1.0" />
-    <xacro:property name="front_ixy" value="0.1" />
-    <xacro:property name="front_ixz" value="0.1" />
-    <xacro:property name="front_iyy" value="0.1" />
-    <xacro:property name="front_iyz" value="0.1" />
-    <xacro:property name="front_izz" value="0.1" />
+    <xacro:property name="front_ixy" value="0.0" />
+    <xacro:property name="front_ixz" value="0.0" />
+    <xacro:property name="front_iyy" value="1.0" />
+    <xacro:property name="front_iyz" value="0.0" />
+    <xacro:property name="front_izz" value="1.0" />
         <!-- steering_link -->
     <xacro:property name="thick_steering" value="0.02" />
     <xacro:property name="alpha" value="${80 * pi / 180}" />
-    <xacro:property name="steering_length" value="${0.2}" />
-    <xacro:property name="mass_steering_link" value="${1.0}" />
+    <xacro:property name="steering_length" value="0.2" />
+    <xacro:property name="mass_steering_link" value="1.0" />
     <xacro:property name="steering_ixx" value="1.0" />
-    <xacro:property name="steering_ixy" value="0.1" />
-    <xacro:property name="steering_ixz" value="0.1" />
-    <xacro:property name="steering_iyy" value="0.1" />
-    <xacro:property name="steering_iyz" value="0.1" />
-    <xacro:property name="steering_izz" value="0.1" />
+    <xacro:property name="steering_ixy" value="0.0" />
+    <xacro:property name="steering_ixz" value="0.0" />
+    <xacro:property name="steering_iyy" value="1.0" />
+    <xacro:property name="steering_iyz" value="0.0" />
+    <xacro:property name="steering_izz" value="1.0" />
         <!-- front wheel  -->
     <xacro:property name="rad_front_wheel" value="${0.216/2}" />
-    <xacro:property name="mass_front_wheel" value="1.0" />
+    <xacro:property name="mass_front_wheel" value="3.0" />
     <xacro:property name="front_ixx" value="1.0" />
-    <xacro:property name="front_ixy" value="0.1" />
-    <xacro:property name="front_ixz" value="0.1" />
-    <xacro:property name="front_iyy" value="0.1" />
-    <xacro:property name="front_iyz" value="0.1" />
-    <xacro:property name="front_izz" value="0.1" />
+    <xacro:property name="front_ixy" value="0.0" />
+    <xacro:property name="front_ixz" value="0.0" />
+    <xacro:property name="front_iyy" value="1.0" />
+    <xacro:property name="front_iyz" value="0.0" />
+    <xacro:property name="front_izz" value="1.0" />
         <!-- back axis -->
     <xacro:property name="length_back_axis" value="0.3" />
     <xacro:property name="rad_back_wheel" value="${0.203/2}" />
         <!-- back wheel inertia -->
-    <xacro:property name="mass_back_wheel" value="1.0" />
+    <xacro:property name="mass_back_wheel" value="1.5" />
     <xacro:property name="back_ixx" value="1.0" />
-    <xacro:property name="back_ixy" value="0.1" />
-    <xacro:property name="back_ixz" value="0.1" />
-    <xacro:property name="back_iyy" value="0.1" />
-    <xacro:property name="back_iyz" value="0.1" />
-    <xacro:property name="back_izz" value="0.1" />
+    <xacro:property name="back_ixy" value="0.0" />
+    <xacro:property name="back_ixz" value="0.0" />
+    <xacro:property name="back_iyy" value="1.0" />
+    <xacro:property name="back_iyz" value="0.0" />
+    <xacro:property name="back_izz" value="1.0" />
 </robot>

File: urdf/test.urdf.xacro (robot description, xacro)
@@ -1,30 +1,74 @@
 <?xml version="1.0"?>
-<robot name="myfirstrobot" xmlns:xacro="http://ros.org/wiki/xacro">
-  <xacro:arg name="use_nominal_extrinsics" default="false"/>
-  <xacro:arg name="add_plug" default="false" />
-  <xacro:arg name="use_mesh" default="true" />
-  <xacro:include filename="$(find realsense2_description)/urdf/_d435.urdf.xacro" />
-  <link name="base_link" />
-  <xacro:sensor_d435 parent="base_link" use_nominal_extrinsics="$(arg use_nominal_extrinsics)" add_plug="1" use_mesh="$(arg use_mesh)">
-    <origin xyz="0 0 0" rpy="0 0 0"/>
-  </xacro:sensor_d435>
-  <xacro:sensor_d435 name="realsense_d435" ropic_ns="realsense_d435" parent="base_link" publish_pointcloud="true">
-    <origin xyz="0.0 0.0 0.0" rpy="0.0 0.0 0.0"/>
-  </xacro:sensor_d435>
-<!--
-  <link name="left_back_wheel_link">
-    <visual>
-      <origin xyz="0 0.11 0"/>
-      <geometry>
-      <mesh filename="package://scooter/meshes/wheel.stl" scale="0.01 0.01 0.01"/>
-        <box size="0.1 0.1 0.1"/>
-      </geometry>
-    </visual>
-  </link>
-  <joint name="base_to_left_back_wheel" type="fixed">
-  	<parent link="base_link"/>
-  	<child link="left_back_wheel_link"/>
-    <origin xyz="0 0.22 0"/>
-  </joint>
--->
+<robot name="scooter" xmlns:xacro="https://www.ros.org/wiki/xacro">
+    <xacro:include filename="$(find autonomous-scooter)/urdf/properties.xacro"/>
+    <link name="base_link">
+        <visual>
+            <geometry>
+                <cylinder length="0.3" radius="0.01"/>
+            </geometry>
+            <origin xyz="0.0 0.0 0.0" rpy="${pi/2} 0.0 0.0"/>
+            <material name='black'/>
+        </visual>
+        <collision>
+            <geometry>
+                <cylinder length="1" radius="0.1"/>
+            </geometry>
+            <origin xyz="0.0 0.0 0.0" rpy="${pi/2} 0.0 0.0"/>
+        </collision>
+        <mass value="${mass_front_wheel}"/>
+        <inertia ixx="${front_ixx}" ixy="${front_ixy}" ixz="${front_ixz}" iyy="${front_iyy}" iyz="${front_iyz}" izz="${front_izz}"/>
+    </link>
+    <!-- front wheel -->
+    <link name="front_wheel_link">
+        <visual>
+            <geometry>
+                <cylinder length="${thick_wheel}" radius="${rad_front_wheel}"/>
+            </geometry>
+            <origin xyz="0.0 0.0 0.0" rpy="${pi/2} 0.0 0.0"/>
+            <material name='black'/>
+        </visual>
+        <collision>
+            <geometry>
+                <cylinder length="${thick_wheel}" radius="${rad_front_wheel}"/>
+            </geometry>
+            <origin xyz="0.0 0.0 0.0" rpy="${pi/2} 0.0 0.0"/>
+        </collision>
+        <mass value="${mass_front_wheel}"/>
+        <inertia ixx="${front_ixx}" ixy="${front_ixy}" ixz="${front_ixz}" iyy="${front_iyy}" iyz="${front_iyz}" izz="${front_izz}"/>
+    </link>
+        <joint name="front_wheel_to_base_joint" type="continuous">
+            <parent link="base_link"/>
+            <child link="front_wheel_link"/>
+            <origin xyz="0.0 0.0 0.0" rpy="0.0 0.0 0.0"/>
+            <axis xyz="0 1 0"/>
+            <limit effort="50" velocity="5.0"/>
+        </joint>
+<!--         <joint name="steering_to_front_joint" type="continuous">
+            <parent link="base_link"/>
+            <child link="base_link"/>
+            <origin xyz="0.0 0.0 ${steering_length/2}" rpy="0.0 0.0 0.0"/>
+            <axis xyz="0 1 0"/>
+            <limit effort="50" velocity="5.0"/>
+        </joint>  -->
+        <transmission name="wheel_motor_transmission">
+            <type>transmission_interface/SimpleTransmission</type>
+            <joint name="front_wheel_to_base_joint">
+                <hardwareInterface>hardware_interface/VelocityJointInterface</hardwareInterface>
+            </joint>
+            <actuator name="wheel_motor">
+                <mechanicalReduction>1</mechanicalReduction>
+            </actuator>
+        </transmission>
+        <gazebo reference="front_wheel_link">
+            <mu1 value="200.0"/>
+            <mu2 value="100.0"/>
+            <kp value="10000000.0" />
+            <kd value="1.0" />>
+        </gazebo>
+    <!-- Gazebo plugin for ROS Control -->
+    <gazebo>
+        <plugin name="gazebo_ros_control" filename="libgazebo_ros_control.so">
+        <robotNamespace>/</robotNamespace>
+        </plugin>
+    </gazebo>
 </robot>
